File: newstuff/UHF_ANTENNA-6U-OFFICIAL-IMPEDANCEMATCHING/UHF_ANTENNA-6U.kicad_pcb (KiCad board)
At the start: 6 copper layers, 206 x 99.1 mm, 47 parts, among them IC1 QBA-07+, IC2 QBA-07+, IC3 QBA-07+, J1 Conn_Coaxial, J2 Conn_01x02, J27 USB_C_Receptacle_USB2.0_16P, J3 Conn_Coaxial, J5 Conn_01x02, J6 Conn_01x02, Q1 IRLML2052, Q27 Q_PMOS_DGS, Q28 Q_PMOS_DGS, U11 CYPD3177-24LQ

Commit message: fix routing
Routing:
- net Net-(IC1-50_OHM_TERM_EXTERNAL): track 0.00 -> 3.16 mm
- net Net-(IC2-50_OHM_TERM_EXTERNAL): track 0.00 -> 3.11 mm
Changed lines of the file:
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@@
 		)
 		(property "Value" "MountingHole"
-			(at 19.046832 58.435555 0)
+			(at -0.221 -4.354 0)
 			(layer "F.Fab")
 			(effects
@@
 	)
 	(segment
+		(start 229.328 54.047)
+		(end 232.418 54.047)
+		(width 0.2)
+		(layer "F.Cu")
+		(net "Net-(IC1-50_OHM_TERM_EXTERNAL)")
+	)
+	(segment
+		(start 232.418 54.047)
+		(end 232.468 53.997)
+		(width 0.2)
+		(layer "F.Cu")
+		(net "Net-(IC1-50_OHM_TERM_EXTERNAL)")
+	)
+	(segment
 		(start 147.320136 66.797)
 		(end 187.700864 66.797)
@@
 	)
 	(segment
+		(start 131.351 70.547)
+		(end 131.358 70.54)
+		(width 0.2)
+		(layer "F.Cu")
+		(net "Net-(IC2-50_OHM_TERM_EXTERNAL)")
+	)
+	(segment
+		(start 128.25 70.547)
+		(end 131.351 70.547)
+		(width 0.2)
+		(layer "F.Cu")
+		(net "Net-(IC2-50_OHM_TERM_EXTERNAL)")
+	)
+	(segment
